Commit message: Added Dependancies in package.xml, modified xacro to modify joint3

File: urdf/robot.xacro (robot description, xacro)
@@ -192,5 +192,5 @@
       <child link="link3"/>
       <axis xyz="0 0 -1"/>
-      <limit effort="1000" lower="-0.3" upper="0.3" velocity="0.1"/>
+      <limit effort="1000" lower="0" upper="1" velocity="0.2"/>
     </joint>
     <gazebo reference="joint3">
@@ -199,5 +199,5 @@
     <link name="link3">
         <visual>
-            <origin xyz="0 0 0" rpy="0 0 0"/>
+            <origin xyz="0 0 ${link_3_length/2}" rpy="0 0 0"/>
             <geometry>
                 <cylinder length="${link_3_length}" radius="${link_3_radius}"/>
@@ -205,5 +205,5 @@
         </visual>
         <collision>
-            <origin xyz="0 0 0" rpy="0 0 0"/>
+            <origin xyz="0 0 ${link_3_length/2}" rpy="0 0 0"/>
             <geometry>
                 <cylinder length="${link_3_length}" radius="${link_3_radius}"/>
@@ -211,5 +211,5 @@
         </collision>
         <inertial>
-            <origin xyz="0 0 0" rpy="0 0 0"/>
+            <origin xyz="0 0 ${link_3_length/2}" rpy="0 0 0"/>
 			<mass value="1"/>
 			<inertia

Commit message: Added Forward Kinematics Code

File: urdf/robot.xacro (robot description, xacro)
@@ -19,4 +19,5 @@
         <parent link="world"/>
         <child link="base_link"/>
+        <origin xyz="0 0 0" rpy="0 0 -1.57"/>
     </joint>
     <link name="base_link">

Commit message: Added Node for Part 2 Plotting part as well as the plots

File: urdf/robot.xacro (robot description, xacro)
@@ -43,5 +43,5 @@
         </inertial>
     </link>
-    <joint name="joint1" type="continuous">
+    <joint name="joint1" type="fixed">
       <!-- <safety_controller k_position="100.0" k_velocity="40.0" soft_lower_limit="-2.8973" soft_upper_limit="2.8973"/> -->
       <origin rpy="0 0 0" xyz="0 0 ${base_link_length}"/>
@@ -50,4 +50,5 @@
       <axis xyz="0 0 1"/>
       <dynamics damping="0.7"/>
+      <!-- <limit effort="1000" lower="-10" upper="10" velocity="50"/> -->
     </joint>
     <link name="link0">
@@ -101,5 +102,5 @@
         </inertial>
     </link>
-    <joint name="joint2" type="revolute">
+    <joint name="joint2" type="fixed">
       <!-- <safety_controller k_position="100.0" k_velocity="40.0" soft_lower_limit="-2.8973" soft_upper_limit="2.8973"/> -->
       <origin rpy="0 0 0" xyz="0 ${link_1_length - unit_radius} 0"/>
@@ -107,5 +108,5 @@
       <child link="joint2link"/>
       <axis xyz="0 0 1"/>
-      <limit effort="1000" lower="-2.8973" upper="2.8973" velocity="2.1750"/>
+      <!-- <limit effort="1000" lower="-2.8973" upper="2.8973" velocity="2.1750"/> -->
     </joint>
     <link name="joint2link">
@@ -193,9 +194,6 @@
       <child link="link3"/>
       <axis xyz="0 0 -1"/>
-      <limit effort="1000" lower="0" upper="1" velocity="0.2"/>
-    </joint>
-    <gazebo reference="joint3">
-      <implicitSpringDamper>1</implicitSpringDamper>
-    </gazebo>
+      <limit effort="10000000" lower="0" upper="1" velocity="2"/>
+    </joint>
     <link name="link3">
         <visual>
@@ -227,28 +225,28 @@
       <minDepth>0.001</minDepth>
     </gazebo> -->
-    <transmission name="tran1">
+    <!-- <transmission name="tran1">
     <type>transmission_interface/SimpleTransmission</type>
     <joint name="joint1">
-      <hardwareInterface>hardware_interface/VelocityJointInterface</hardwareInterface>
+      <hardwareInterface>EffortJointInterface</hardwareInterface>
     </joint>
     <actuator name="motor1">
-      <hardwareInterface>hardware_interface/VelocityJointInterface</hardwareInterface>
+      <hardwareInterface>EffortJointInterface</hardwareInterface>
       <mechanicalReduction>1</mechanicalReduction>
     </actuator>
-  </transmission>
-  <transmission name="tran2">
+  </transmission> -->
+  <!-- <transmission name="tran2">
     <type>transmission_interface/SimpleTransmission</type>
     <joint name="joint2">
-      <hardwareInterface>hardware_interface/VelocityJointInterface</hardwareInterface>
+      <hardwareInterface>EffortJointInterface</hardwareInterface>
     </joint>
     <actuator name="motor2">
-      <hardwareInterface>hardware_interface/VelocityJointInterface</hardwareInterface>
+      <hardwareInterface>EffortJointInterface</hardwareInterface>
       <mechanicalReduction>1</mechanicalReduction>
     </actuator>
-  </transmission>
+  </transmission> -->
   <transmission name="tran3">
       <type>transmission_interface/SimpleTransmission</type>
       <joint name="joint3">
-	<hardwareInterface>hardware_interface/VelocityJointInterface</hardwareInterface>
+	<hardwareInterface>EffortJointInterface</hardwareInterface>
       </joint>
       <actuator name="motor3">
@@ -256,6 +254,6 @@
       </actuator>
     </transmission>
-    <gazebo reference="joint3">
+    <!-- <gazebo reference="joint3">
       <implicitSpringDamper>1</implicitSpringDamper>
-    </gazebo>
+    </gazebo> -->
 </robot>

Commit message: Added Time Measurement Logic

File: urdf/robot.xacro (robot description, xacro)
@@ -50,5 +50,5 @@
       <axis xyz="0 0 1"/>
       <dynamics damping="0.7"/>
-      <!-- <limit effort="1000" lower="-10" upper="10" velocity="50"/> -->
+      <limit effort="1000" lower="-10" upper="10" velocity="2.1750"/>
     </joint>
     <link name="link0">
@@ -108,5 +108,5 @@
       <child link="joint2link"/>
       <axis xyz="0 0 1"/>
-      <!-- <limit effort="1000" lower="-2.8973" upper="2.8973" velocity="2.1750"/> -->
+      <limit effort="1000" lower="-2.8973" upper="2.8973" velocity="2.1750"/>
     </joint>
     <link name="joint2link">
@@ -194,5 +194,5 @@
       <child link="link3"/>
       <axis xyz="0 0 -1"/>
-      <limit effort="10000000" lower="0" upper="1" velocity="2"/>
+      <limit effort="1000" lower="0" upper="1" velocity="2"/>
     </joint>
     <link name="link3">
@@ -211,5 +211,5 @@
         <inertial>
             <origin xyz="0 0 ${link_3_length/2}" rpy="0 0 0"/>
-			<mass value="1"/>
+			<mass value="0.1"/>
 			<inertia
 			  ixx="${mass/12*(3*link_3_radius*link_3_radius + link_3_length*link_3_length)}" ixy="0.0" ixz="0.0"
@@ -244,6 +244,6 @@
       <mechanicalReduction>1</mechanicalReduction>
     </actuator>
-  </transmission> -->
-  <transmission name="tran3">
+  </transmission>  -->
+   <transmission name="tran3">
       <type>transmission_interface/SimpleTransmission</type>
       <joint name="joint3">

Commit message: Final Push

File: urdf/robot.xacro (robot description, xacro)
@@ -43,5 +43,5 @@
         </inertial>
     </link>
-    <joint name="joint1" type="fixed">
+    <joint name="joint1" type="continuous">
       <!-- <safety_controller k_position="100.0" k_velocity="40.0" soft_lower_limit="-2.8973" soft_upper_limit="2.8973"/> -->
       <origin rpy="0 0 0" xyz="0 0 ${base_link_length}"/>
@@ -102,5 +102,5 @@
         </inertial>
     </link>
-    <joint name="joint2" type="fixed">
+    <joint name="joint2" type="revolute">
       <!-- <safety_controller k_position="100.0" k_velocity="40.0" soft_lower_limit="-2.8973" soft_upper_limit="2.8973"/> -->
       <origin rpy="0 0 0" xyz="0 ${link_1_length - unit_radius} 0"/>
@@ -225,30 +225,31 @@
       <minDepth>0.001</minDepth>
     </gazebo> -->
-    <!-- <transmission name="tran1">
+    <transmission name="tran1">
     <type>transmission_interface/SimpleTransmission</type>
     <joint name="joint1">
-      <hardwareInterface>EffortJointInterface</hardwareInterface>
+      <hardwareInterface>hardware_interface/EffortJointInterface</hardwareInterface>
     </joint>
     <actuator name="motor1">
-      <hardwareInterface>EffortJointInterface</hardwareInterface>
+    <hardwareInterface>hardware_interface/EffortJointInterface</hardwareInterface>
       <mechanicalReduction>1</mechanicalReduction>
     </actuator>
-  </transmission> -->
-  <!-- <transmission name="tran2">
+  </transmission>
+  <transmission name="tran2">
     <type>transmission_interface/SimpleTransmission</type>
     <joint name="joint2">
-      <hardwareInterface>EffortJointInterface</hardwareInterface>
+      <hardwareInterface>hardware_interface/EffortJointInterface</hardwareInterface>
     </joint>
     <actuator name="motor2">
-      <hardwareInterface>EffortJointInterface</hardwareInterface>
+    <hardwareInterface>hardware_interface/EffortJointInterface</hardwareInterface>
       <mechanicalReduction>1</mechanicalReduction>
     </actuator>
-  </transmission>  -->
+  </transmission>
    <transmission name="tran3">
       <type>transmission_interface/SimpleTransmission</type>
       <joint name="joint3">
-	<hardwareInterface>EffortJointInterface</hardwareInterface>
+	<hardwareInterface>hardware_interface/EffortJointInterface</hardwareInterface>
       </joint>
       <actuator name="motor3">
+      <hardwareInterface>hardware_interface/EffortJointInterface</hardwareInterface>
 	<mechanicalReduction>1</mechanicalReduction>
       </actuator>
